File: Macropad.kicad_sch (KiCad schematic)
At the start: 11 parts, among them SW1 SW_Push, SW2 SW_Push, SW3 SW_Push, SW4 SW_Push, SW5 SW_Push, U1 XIAO-RP2040-DIP

Commit message: added the libraries!!!
Parts:
- removed OL1: OLED, display:SSD1306_OLED-0.91-128x32, symbol oled:OLED
- added D5: SK6812MINI, LED_SMD:LED_SK6812MINI_PLCC4_3.5x3.5mm_P1.75mm, symbol LED:SK6812MINI
- added J1: Conn_01x04, display:SSD1306-0.91-OLED-4pin-128x32, symbol Connector_Generic:Conn_01x04
Connections:
- net +5V: now also D5.4 (VDD), J1.2 (Pin_2)
- net GND: now also D5.2 (VSS), J1.1 (Pin_1)
- net at U1.2 (GPIO27/ADC1/A1): now also J1.3 (Pin_3)
- net at U1.1 (GPIO26/ADC0/A0): now also J1.4 (Pin_4)
- net at D4.1 (DOUT): now also D5.3 (DIN)
Other:
- moved on the sheet: D3, D4
