File: PCB/Macropad.kicad_pcb (KiCad board)
At the start: 2 copper layers, 100 x 63.9 mm, 12 parts, among them J1 Conn_01x04, SW1 SW_Push, SW2 SW_Push, SW3 SW_Push, SW4 SW_Push, SW5 SW_Push, U1 XIAO-RP2040-DIP

Commit message: Organized the files
Routing:
- net GND: track 316.7 -> 324.5 mm
Other:
- board text added: "Macropad by BedTime"
- board text added: "macropad by BedTime"
Changed lines of the file:
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@@
 		(layer "Edge.Cuts")
+	)
+	(gr_text "macropad by BedTime"
+		(at 188 190 0)
+		(layer "F.Cu")
+		(effects
+			(font
+				(size 1.5 1.5)
+				(thickness 0.3)
+				(bold yes)
+			)
+			(justify left bottom)
+		)
+	)
+	(gr_text "Macropad by BedTime"
+		(at 122 121 0)
+		(layer "F.SilkS")
+		(effects
+			(font
+				(size 1 1)
+				(thickness 0.25)
+				(bold yes)
+			)
+			(justify left bottom)
+		)
 	)
 	(gr_text "　　　　　　 　 　 　 　 /　/　,　-‐─‐- ..__／'￣｀ 　 ＿\n　　　　　　　　 ,　-‐ｧ′/／／　￣￣｀　//⌒＝ミ,　| | |\n　　　　　 　 ／　　./　 / ／　　　　　　　　　 ⌒＼＼| | |\n　　　　　　/　　　.::| 　｛//　　　　 ／　　　　　　　 ＼ｉ | |\n.　　　　　/　　 .:　.:|　〃　　　　／　 ／／　　 j 　 　 | | |\n　　　　　′　 .:　.::｣_//　　　／ ,_／／〃　　 /　　　i∨ハ\n　　　　 i　　　:　.:|　Y{　　〃__彡'＾く／/　　//ii　i 　 ! |(　 ∨ /\n　　　　 !　　 　 .::|||l.|｢　//ｨﾃそk 彡 /　／_⌒|　!　 j :| ｀.　∨ /\n.　　 　 i　　　　　|__/|: //|弋ｚｿ　　／イｯ'てトJ /　/} ハ :　 ∨ /\n.　　 　 |　　　 　 :.:.V|/V｜　　　　　　　ヒ ｿ ﾉj/　/ｨ/　 '.　　 ∨ /\n.　　 　 |　　　 　 :.:.:!i|l「ﾍ.ﾄ,　　 ､　　　' __　　〃 〃/{　:.　:　　 i∨\n.　　 　 |　　　　　:.:.:.:|!ﾏ={{ ＼　 ＿ｰ‐ |ｉｉ| .ｲ / /イ{｛　:.　:.　　 i'.　/\n.　　 　 |　　　　　 :.:.:.Vﾊ　＼/{h.ﾏﾊ - |ｉｉ｢／7/^'くj {　 　 　 　 i ∨\n.　　 　 |　　　　　 　 :.:Vﾊ.　 { {|:　ﾏﾊ　|ｉｉ|{　/'　 　 V:　　　　　 i. '.　/\n　 　 　 !.　　　　　　　.:.V＞'7　＼/ﾏ|,//ﾊ　　 　 　 i:　　　:. :　 i.　∨ /\n　 　 　 i:　　　　　　/　　　 /|　/＾＼V//ハ 　 []｜ |: : .　: : :　 i 　 ∨\n　　　　 !:.　　　　　 i 　 　 ￡|/ 》‐｢＾}ｉｉi|　　ｉ　　　　,^ : :. .: .:　　i\n　　　　 i :　　 　 　 |　　　￡ 　 |　|　|ｉｉi|　　|＿＿__ji　:. : .:　.\n　　　　 | :　　 　 　 |　　 V　 　 |　|　|　|　 ｢|￣￣[_,|:　: : .:　:.\n　　　　 | :.　　　 　 :! 　 /　　　｜ |　|　|　 |:|　　 　:||i　: :　:.　:"
@@
 	)
 	(segment
+		(start 158.152 71.452)
+		(end 149.86469 71.452)
+		(width 0.2)
+		(layer "F.Cu")
+		(net 1)
+	)
+	(segment
+		(start 91.101 92.849)
+		(end 90 93.95)
+		(width 0.2)
+		(layer "F.Cu")
+		(net 1)
+	)
+	(segment
 		(start 115.65 114.275)
 		(end 115.65 125.54)
@@
 	)
 	(segment
-		(start 158.152 71.452)
-		(end 149.86469 71.452)
-		(width 0.2)
-		(layer "F.Cu")
-		(net 1)
-	)
-	(segment
-		(start 91.101 92.849)
-		(end 90 93.95)
+		(start 113.349 111.974)
+		(end 115.65 114.275)
 		(width 0.2)
 		(layer "F.Cu")
@@
 	)
 	(segment
+		(start 113.349 108.926)
+		(end 113.349 111.974)
+		(width 0.2)
+		(layer "F.Cu")
+		(net 1)
+	)
+	(segment
 		(start 96.735 125.54)
 		(end 95.73 125.54)
@@
 		(width 0.2)
 		(layer "F.Cu")
+		(net 1)
+	)
+	(segment
+		(start 114.45 107.825)
+		(end 113.349 108.926)
+		(width 0.2)
+		(layer "F.Cu")
