File: PCB/Macropad.kicad_sch (KiCad schematic)
At the start: 12 parts, among them J1 Conn_01x04, SW1 SW_Push, SW2 SW_Push, SW3 SW_Push, SW4 SW_Push, SW5 SW_Push, U1 XIAO-RP2040-DIP

Commit message: Organized the files
Other:
- note added: "macropad by BedTime"
Changed lines of the file:
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@@
 	(generator_version "9.0")
 	(paper "A4")
+	(text "macropad by BedTime"
+		(exclude_from_sim no)
+		(at 197.866 189.484 0)
+		(effects
+			(font
+				(size 1.27 1.27)
+			)
+		)
+	)
 	(junction
 		(at 113.03 124.46)
